Commit message: make it look nicer

File: sapien_franka/panda.urdf (robot description, URDF)
Before this commit: robot panda, 12 links, 11 joints
Links:
- link panda_hand: geometry collision mesh filename=franka_description/meshes/collision/hand.stl; visual mesh filename=franka_description/meshes/visual/hand.glb
- link panda_leftfinger: geometry collision mesh filename=franka_description/meshes/collision/finger.stl; visual mesh filename=franka_description/meshes/visual/finger.glb
- link panda_link0: geometry collision mesh filename=franka_description/meshes/collision/link0.stl; visual mesh filename=franka_description/meshes/visual/link0.glb
- link panda_link1: geometry collision mesh filename=franka_description/meshes/collision/link1.stl; visual mesh filename=franka_description/meshes/visual/link1.glb
- link panda_link2: geometry collision mesh filename=franka_description/meshes/collision/link2.stl; visual mesh filename=franka_description/meshes/visual/link2.glb
- link panda_link3: geometry collision mesh filename=franka_description/meshes/collision/link3.stl; visual mesh filename=franka_description/meshes/visual/link3.glb
- link panda_link4: geometry collision mesh filename=franka_description/meshes/collision/link4.stl; visual mesh filename=franka_description/meshes/visual/link4.glb
- link panda_link5: geometry collision mesh filename=franka_description/meshes/collision/link5.stl; visual mesh filename=franka_description/meshes/visual/link5.glb
- link panda_link6: geometry collision mesh filename=franka_description/meshes/collision/link6.stl; visual mesh filename=franka_description/meshes/visual/link6.glb
- link panda_link7: geometry collision mesh filename=franka_description/meshes/collision/link7.stl; visual mesh filename=franka_description/meshes/visual/link7.glb
- link panda_rightfinger: geometry collision mesh filename=franka_description/meshes/collision/finger.stl; visual mesh filename=franka_description/meshes/visual/finger.glb
